File: UHF-PCB-6layer/UHF-PCB-6layer.kicad_pcb (KiCad board)
At the start: 2 copper layers, 34 parts, among them J1 Screw_Terminal_01x07, J2 Screw_Terminal_01x04, U1 MAC-24+, U2 LTC1566-1IS8-PBF, U3 TAV1-331+, U4 MAC-24+, U5 XMSM0G3507SPT, U6 XC7A100T-CSG324_A, U7 MC100EL1648DTR2G

Commit message: started layout for PCB
Parts:
- moved U6 116.8 mm to (30.2, 66.6)
- moved J1 115.6 mm to (21.1, 127.3)
- moved U5 113.4 mm to (29.0, 26.7)
- moved U7 100.6 mm to (62.5, 41.1)
- moved D1 100.6 mm to (60.9, 44.8)
- moved U3 100.6 mm to (64.9, 45.1)
- moved CR1 91.0 mm to (55.3, 31.9)
- moved U2 91.0 mm to (55.3, 38.5)
- moved C1 88.0 mm to (34.1, 37.1)
- moved C10 88.0 mm to (38.1, 42.1)
- moved C2 88.0 mm to (34.1, 39.6)
- moved C3 88.0 mm to (34.1, 42.1)
- moved C4 88.0 mm to (34.1, 44.6)
- moved C5 88.0 mm to (34.1, 47.2)
- moved C6 88.0 mm to (34.1, 49.7)
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